Commit message: [fix] 射出機構: 射出輪に摩擦を与え、食い込みを 10 mm から 1 mm へ
ディスクがほとんど発射されず、20 発撃っても 19 発が足元に落ちていた。まれに
出る 1 発も 350 m 飛ぶなど、同じ指令で挙動がまったく揃わなかった。

原因は 2 つある。

1. 射出輪の衝突マテリアルが shooter_unit (dynamic 0.0, combine minimum) だった。
   これは通路の壁がディスクを引っ掛けないための低摩擦指定で、掴む側に使うもの
   ではない。フライホイール式は摩擦で送り出す機構なので、接線力が原理的に
   発生しない。まれに飛んでいたのは下の食い込みによる法線方向の力積で、
   方向も速度も制御されていなかった。

2. 射出輪の内面間隔が 0.16 m で、ディスク直径 0.18 m に対して片側 10 mm 貫入
   していた。剛体どうしでこれだけ食い込むと解消時に過大な力積が出る。あわせて
   質量 10 kg・慣性 1.0 という、半径 4 cm の円盤としてありえない値が入っていて
   (izz = m r^2 / 2 なら 0.008)、反力を受け流さないぶん力積を増幅していた。

射出輪だけ shooter_roller (static 1.0, dynamic 0.9, combine maximum) にした。
maximum は minimum より優先されるので、ディスク側が dynamic 0.1 の minimum でも
この値が効く。壁は shooter_unit のままなので引っ掛かりは増えない。食い込みは
片側 1 mm、質量は 0.5 kg、慣性は形状から算出した値にした。接線力には法線力が
要るので食い込みを 0 にはしない。

諸元は xacro プロパティにまとめたので、以後の調整は roller_squeeze など 1 行で
済む。

実測 (ロボットは動かさず 20 発、200 Hz):
  発射率        1/20 -> 20/20
  飛距離        ばらばら (足元〜350 m) -> 中央値 12.8 m
  2 m の標的    命中せず -> 命中、HP 200 -> 190、装甲板 1 が反応

残る制約: 約 4 度の右偏りがある。2.0 m では当たるが 2.5 m では 0.1〜0.2 m 右へ
外れる。装甲板が 0.15 m 角と小さいので距離が伸びるほど当てにくい。射出輪の配置は
左右対称で逆回転も正しいため、原因は未特定。

Co-Authored-By: Claude Opus 5 (1M context) <noreply@anthropic.com>

File: colcon_ws/src/sample_robot_description/urdf/common.xacro (robot description, xacro)
@@ -23,4 +23,14 @@
     <collision_material name="shooter_unit">
       <friction static="0.2" dynamic="0.0" combine="minimum"/>
+    </collision_material>
+    <!--
+      射出輪だけは掴む側。ディスクの材質は dynamic 0.1 の minimum なので、
+      こちらを minimum のままにすると接線力がまったく出ず、フライホイール式の
+      射出が成立しない (ディスクは輪をすり抜けて足元に落ちる)。maximum は
+      minimum より優先されるので、ディスク側の指定に関わらずこの値が効く。
+      通路の壁は shooter_unit のままなので、引っ掛かりは増えない。
+    -->
+    <collision_material name="shooter_roller">
+      <friction static="1.0" dynamic="0.9" combine="maximum"/>
     </collision_material>
   </xacro:macro>

File: colcon_ws/src/sample_robot_description/urdf/shooter/shooter.urdf.xacro (robot description, xacro)
@@ -1,4 +1,33 @@
 <?xml version="1.0"?>
 <robot xmlns:xacro="http://ros.org/wiki/xacro">
+  <!--
+    射出輪の諸元。ここだけ触れば噛み具合を調整できる。
+    disc_radius        ディスクの半径 (flying_disc_description と揃えること)
+    roller_radius      射出輪の半径
+    roller_width       射出輪の厚み。ディスクの厚み 0.02 より広く取り、
+                       ディスクが上下にずれても外れないようにする
+    roller_squeeze     片側あたりの食い込み量。射出輪の間隔はこれで決まる:
+                         y = ±(disc_radius + roller_radius - roller_squeeze)
+    roller_squeeze は 0.001 にしてある。以前は射出輪の中心が y = ±0.12、
+    半径 0.04 で内面が ±0.08、ディスク直径 0.18 に対して片側 10 mm も
+    食い込んでいた。剛体どうしでこれだけ貫入すると解消時に過大な力積が出て、
+    同じ指令でも足元に落ちる弾と 350 m 飛ぶ弾が混ざる。接線力で送り出すには
+    法線力が要るので 0 にはせず、わずかに噛ませる。
+  -->
+  <xacro:property name="disc_radius"   value="0.09"/>
+  <xacro:property name="roller_radius" value="0.04"/>
+  <xacro:property name="roller_width"  value="0.03"/>
+  <xacro:property name="roller_squeeze" value="0.001"/>
+  <xacro:property name="roller_offset"
+                  value="${disc_radius + roller_radius - roller_squeeze}"/>
+  <!-- 実体に見合った慣性。以前は質量 10 kg・慣性 1.0 で、半径 0.04 の円盤として
+       ありえない値だった (izz = m r^2 / 2 なら 0.008)。慣性が過大なぶん食い込みの
+       反力を一切受け流さず、上の力積を増幅していた。800 rad/s での回転エネルギは
+       この値でも 1 発 (7.7 J) に対して十分余裕がある。 -->
+  <xacro:property name="roller_mass"   value="0.5"/>
+  <xacro:property name="roller_izz"
+                  value="${0.5 * roller_mass * roller_radius * roller_radius}"/>
+  <xacro:property name="roller_ixx"
+                  value="${roller_mass * (3 * roller_radius * roller_radius + roller_width * roller_width) / 12.0}"/>
   <xacro:macro name="shooter_v0" params="parent *joint_origin">
         <joint name="shooter_shaft_link_joint" type="fixed">
@@ -409,5 +438,5 @@
         </link>
          <joint name="shooter_wheel1_link_joint" type="continuous">
-          <origin rpy="0 0 0" xyz="0.15 0.12 0.055"/> <!-- disc pos x 0.18 z -0.0925 -->
+          <origin rpy="0 0 0" xyz="0.15 ${roller_offset} 0.055"/>
           <parent link="shooter_base_link"/>
           <child link="shooter_wheel1_link"/>
@@ -420,24 +449,26 @@
           <visual>
                 <geometry>
-                  <cylinder length="0.02" radius="0.04" />
+                  <cylinder length="${roller_width}" radius="${roller_radius}" />
                 </geometry>
                 <material name="gray"/>
           </visual>
           <collision>
-            <collision_material name="shooter_unit"/>
-                <geometry>
-                  <cylinder length="0.02" radius="0.04" />
-                </geometry>
-          </collision>
-          <inertial>
-                <origin xyz="0 0 0"/>
-                <mass value="10.0"/>
-                <inertia ixx="1" ixy="0" ixz="0"
-                                 iyy="1" iyz="0"
-                                 izz="1" />
+            <!-- 射出輪だけは掴む側。shooter_unit (dynamic 0, combine minimum) の
+                 ままだと接線力が出ず、フライホイール式として成立しない。 -->
+            <collision_material name="shooter_roller"/>
+                <geometry>
+                  <cylinder length="${roller_width}" radius="${roller_radius}" />
+                </geometry>
+          </collision>
+          <inertial>
+                <origin xyz="0 0 0"/>
+                <mass value="${roller_mass}"/>
+                <inertia ixx="${roller_ixx}" ixy="0" ixz="0"
+                                 iyy="${roller_ixx}" iyz="0"
+                                 izz="${roller_izz}" />
           </inertial>
         </link>
          <joint name="shooter_wheel2_link_joint" type="continuous">
-          <origin rpy="0 0 0" xyz="0.15 -0.12 0.055"/> <!-- disc pos x 0.18 z -0.0925 -->
+          <origin rpy="0 0 0" xyz="0.15 ${-roller_offset} 0.055"/>
           <parent link="shooter_base_link"/>
           <child link="shooter_wheel2_link"/>
@@ -450,20 +481,20 @@
           <visual>
                 <geometry>
-                  <cylinder length="0.02" radius="0.04" />
+                  <cylinder length="${roller_width}" radius="${roller_radius}" />
                 </geometry>
                 <material name="gray"/>
           </visual>
           <collision>
-            <collision_material name="shooter_unit"/>
-                <geometry>
-                  <cylinder length="0.02" radius="0.04" />
-                </geometry>
-          </collision>
-          <inertial>
-                <origin xyz="0 0 0"/>
-                <mass value="10.0"/>
-                <inertia ixx="1" ixy="0" ixz="0"
-                                 iyy="1" iyz="0"
-                                 izz="1" />
+            <collision_material name="shooter_roller"/>
+                <geometry>
+                  <cylinder length="${roller_width}" radius="${roller_radius}" />
+                </geometry>
+          </collision>
+          <inertial>
+                <origin xyz="0 0 0"/>
+                <mass value="${roller_mass}"/>
+                <inertia ixx="${roller_ixx}" ixy="0" ixz="0"
+                                 iyy="${roller_ixx}" iyz="0"
+                                 izz="${roller_izz}" />
           </inertial>
         </link>

Commit message: [add] contact_offset は見かけの半径として効く。間隔と連動させる
contact_offset を振って過速の弾を減らせないか調べる過程で、この値が
「接触を生成し始める距離」以上の働きをすることが分かった。

0.02 にしたうえで射出輪の間隔を +0.01 広げ、幾何的には 8 mm の隙間が空く配置に
しても、20 発すべてが 31〜36 m/s で発射された。触れていないのに駆動されている
以上、殻の厚みぶん太った円柱として振る舞っている。間隔をそのままで値だけ広げると
実効的な食い込みが増えるので、roller_offset に既定 0.01 からの増分を足して
相殺するようにした。roller_contact_offset は common.xacro に置き、材質と間隔の
両方から参照する。

値そのものは既定 (0.01) のままにしてある。挙動は従来と変わらない。

過速の弾 (38〜100 m/s) の削減は決着しなかった。20 発ずつの測定で:

  0.01 (既定)      方位の中央値 +0.57 度、正常な弾 -0.21〜+0.64 度、過速 4/20
  0.02 + 間隔補正  1 回目 -0.11 度 / -0.89〜+0.21 度、2 回目 +0.72 度 /
                   -0.27〜+2.94 度
  0.03 + 間隔補正  悪化 (弱い弾が増え、過速も 6/15)

0.02 が良く見えた回があり、系統的な右偏りも消えたように見えたが、まわし直すと
再現しなかった。回ごとの差が設定間の差より大きく、1 回ずつでは判定できない。
判定するなら各設定で複数回まわすこと。

Co-Authored-By: Claude Opus 5 (1M context) <noreply@anthropic.com>

File: colcon_ws/src/sample_robot_description/urdf/common.xacro (robot description, xacro)
@@ -11,4 +11,7 @@
     逆に低摩擦を効かせたいシュータ内部は minimum です。
   -->
+  <!-- 射出輪の contact_offset。Unity の既定は 0.01。shooter.urdf.xacro が
+       射出輪の間隔を決めるときにも参照する (増分だけ間隔を広げて相殺する)。 -->
+  <xacro:property name="roller_contact_offset" value="0.01"/>
   <xacro:macro name="sample_robot_collision_materials">
     <!-- 車輪のバレル: 床をつかむ側。指定値を確実に効かせる -->
@@ -33,14 +36,19 @@
     <collision_material name="shooter_roller">
       <friction static="1.0" dynamic="0.9" combine="maximum"/>
+      <contact_offset value="${roller_contact_offset}"/>
       <!--
-        contact_offset (既定 0.01) を広げると、幾何的に重なる前から接触が生成され、
-        食い込みを一気に解消するときの力積が和らぐ。20 発ずつ測った結果:
-          未設定    正常な弾の方位 -0.21〜+0.64 度、ただし 4/20 が 38〜100 m/s の
-                    過速で ±22〜27 度へ飛ぶ
-          0.02      過速は消える (最大 42 m/s)。かわりに正常な弾の方位が
-                    -0.11〜+5.22 度へ広がる
-        どちらを取るかは決めきれていないので、既定のままにしてある。2.5 m の標的への
-        命中数でも比べたが、同じ設定でも 2 発命中する回と 0 発の回があり、1 回ずつの
-        試行では設定の優劣を判定できない。判断するなら各設定で複数回まわすこと。
+        contact_offset は「接触を生成し始める距離」だが、実測では見かけの半径として
+        振る舞う。0.02 にして射出輪の間隔を +0.01 広げ、幾何的には 8 mm の隙間が
+        空く配置にしても、20 発すべてが 31〜36 m/s で発射された。触れていないのに
+        駆動されている以上、殻の厚みぶん太った円柱として効いている。値を変えるなら
+        shooter.urdf.xacro の roller_offset で間隔を補正すること (相殺済み)。
+        過速で飛ぶ弾 (38〜100 m/s) を減らせないかと値を振ってみたが、決着していない。
+        20 発ずつの測定で:
+          0.01 (既定)      方位の中央値 +0.57 度、正常な弾 -0.21〜+0.64 度、過速 4/20
+          0.02 + 間隔補正  1 回目 -0.11 度 / -0.89〜+0.21 度、2 回目 +0.72 度 /
+                           -0.27〜+2.94 度。回ごとの差が設定間の差より大きい
+          0.03 + 間隔補正  悪化 (弱い弾が増え、過速も 6/15 に増える)
+        0.02 が良く見えた回もあるが再現しない。判定するなら各設定で複数回まわすこと。
+        既定のままにしてある。
       -->
     </collision_material>

File: colcon_ws/src/sample_robot_description/urdf/shooter/shooter.urdf.xacro (robot description, xacro)
@@ -32,6 +32,14 @@
   <xacro:property name="wall_length" value="0.22"/>
   <xacro:property name="wall_center_x" value="0.01"/>
+  <!--
+    間隔には roller_contact_offset (common.xacro で定義) の増分も足す。
+    contact_offset は接触を生成し始める距離なので、大きくすると触れる前から
+    投機的接触で速度が制限され、見かけ上ローラーが太ったように振る舞う。間隔を
+    そのままで広げると実効的な食い込みが増えるため、既定 0.01 からの増分だけ
+    間隔を広げて相殺する。
+  -->
   <xacro:property name="roller_offset"
-                  value="${disc_radius + roller_radius - roller_squeeze}"/>
+                  value="${disc_radius + roller_radius - roller_squeeze
+                          + (roller_contact_offset - 0.01)}"/>
   <!-- 実体に見合った慣性。以前は質量 10 kg・慣性 1.0 で、半径 0.04 の円盤として
        ありえない値だった (izz = m r^2 / 2 なら 0.008)。慣性が過大なぶん食い込みの
