Commit message: [fix] シミュレータ v1.0.3 対応と、実機評価で見つかった駆動系の不具合
シミュレータ:
- SIMULATOR_VERSION / 実行ファイルのパスを v1.0.3 へ
- launch_docker.sh に WSLg の GPU 受け渡しを追加。/dev/dxg があっても
  コンテナには /dev/dri が現れず、Mesa が llvmpipe (ソフトウェア描画) を
  選んでしまうため GALLIUM_DRIVER=d3d12 も明示する。

ロボットが動かない問題:
- 関節に <drive> が無く、指令が届いても回っていなかった。Unity 版は
  URDF-Importer の <drive stiffness= damping=> を ArticulationDrive に
  当てる方式で、Isaac 用の <isaac_drive_api> は読まれない。駆動輪・
  シュータの各関節へ追加した。<drive> を外すと機体が不安定になり転倒する。
- <limit> も無かったので forceLimit / maxJointVelocity が既定のままだった。
  ros2_control の指令上限 (射出輪 1600 rad/s、装填 6) に合わせた。
  フリーローラ側は逆に上げすぎると 1 ステップの回転量が過大になり接触が
  壊れるため 100 に抑える。

オムニホイールが空転する問題:
- 物理レート既定 50 Hz では接地しているフリーローラ (直径約 3 cm) の
  接触が保てず、0.4 m/s 指令に対し 0.127 m/s (32%) しか出ていなかった。
  settings.physics_hz=200 の simulation_resources.json を追加し、
  bring_up から SIMULATION_RESOURCES_CONFIG で渡す。
  200 Hz で 0.242 m/s (61%)、RTF は 0.56 -> 0.57 でほぼ変わらない。

Co-Authored-By: Claude Opus 5 (1M context) <noreply@anthropic.com>

File: colcon_ws/src/sample_robot_description/urdf/shooter/shooter.urdf.xacro (robot description, xacro)
@@ -378,5 +378,7 @@
          <joint name="shooter_loader_link_joint" type="prismatic">
           <origin rpy="0 0 0" xyz="-0.12 0 0.05"/>
-          <limit lower="0.0" upper="0.2" effort="100" velocity="1.0" />
+          <limit lower="0.0" upper="0.2" effort="100" velocity="10.0" />
+          <!-- Unity: 装填機構。ros2_control の指令上限は 6 なので velocity もそれ以上に取る -->
+          <drive stiffness="0.0" damping="30000.0"/>
           <parent link="shooter_base_link"/>
           <child link="shooter_loader_link"/>
@@ -411,4 +413,7 @@
           <child link="shooter_wheel1_link"/>
           <axis xyz="0 0 1"/>
+          <!-- Unity: 射出輪。ros2_control の指令上限 1600 rad/s に合わせる -->
+          <drive stiffness="0.0" damping="100.0"/>
+          <limit effort="100.0" velocity="2000.0"/>
         </joint>
         <link name="shooter_wheel1_link">
@@ -438,4 +443,7 @@
           <child link="shooter_wheel2_link"/>
           <axis xyz="0 0 -1"/>
+          <!-- Unity: 射出輪。ros2_control の指令上限 1600 rad/s に合わせる -->
+          <drive stiffness="0.0" damping="100.0"/>
+          <limit effort="100.0" velocity="2000.0"/>
         </joint>
         <link name="shooter_wheel2_link">

File: colcon_ws/src/sample_robot_description/urdf/wheel/wheel_100mm.urdf.xacro (robot description, xacro)
@@ -8,4 +8,10 @@
       <axis xyz="0 0 1"/>
       <isaac_drive_api stiffness="0" damping="0" joint_friction="0"/>
+      <!-- Unity: フリーローラなので駆動なし (Isaac の damping=0 と同じ意味)。
+           <limit velocity> は maxJointVelocity になる。既定 (100) より上げると
+           50 Hz の物理刻みでは 1 ステップの回転量が大きくなりすぎて接触が壊れる。
+           ローラは車体 0.6 m/s でも 40 rad/s 程度なので 100 で足りる。 -->
+      <drive stiffness="0.0" damping="0.0"/>
+      <limit effort="0.0" velocity="100.0"/>
     </joint>
     <link name="${prefix}_link">
@@ -35,4 +41,8 @@
     <axis xyz="0 0 1"/>
     <isaac_drive_api stiffness="0" damping="30000" joint_friction="0"/>
+    <!-- Unity: 速度制御用のドライブ。<isaac_drive_api> は Isaac 専用で
+         こちらは読まれないため、同じ意味の <drive> を併記する。 -->
+    <drive stiffness="0.0" damping="30000.0"/>
+    <limit effort="100.0" velocity="100.0"/>
   </joint>
     <link name="${prefix}_housing_link">

Commit message: [fix] 射出機構: 通路の遊びを詰め、噛み位置まで案内する
右偏りの原因を調べた。飛翔中の弾の速度ベクトル (EntityState.twist) を読むと、
射出は 2 つの群に分かれていた。

  両輪で噛んだ弾  33〜35 m/s、方位 +0.3〜+1.2 度
  片輪だけの弾    10〜18 m/s、方位 -12〜+14 度

偏りそのものより、片輪だけで蹴られる弾が半数あることが問題だった。駆動が
半分になるうえ横向きの力が残る。

通路の壁の内面が ±0.10、ディスク半径 0.09 で片側 10 mm の遊びがあり、食い込みは
片側 1 mm しかなかった。遊びの範囲で寄れば反対側の輪には届かない。壁の x 範囲も
-0.10〜+0.10 で、射出輪の前縁 0.11 に届いておらず、噛む直前が無案内だった。

遊びを 1.5 mm に詰め、食い込みを 2 mm に増やし (最悪の寄りでも反対側に 0.5 mm
触れる)、壁を x=+0.12 まで延ばした。壁の位置と長さも xacro プロパティにした。

実測 (20 発、速度ベクトルから方位を算出):
  方位の中央値          +1.55 度 -> +0.57 度
  両輪で噛んだ弾の方位  +0.34〜+1.15 度 -> -0.21〜+0.64 度
  片輪だけの弾の方位    -12.1〜+13.9 度 -> +0.5〜+1.9 度
  2.5 m の標的          命中せず -> 2 発命中、HP 200 -> 180、装甲板 1 と 2 が反応

遊びを 0.5 mm、食い込みを 1 mm まで詰める案も試したが悪化した (捉えた弾が 20 発
から 13 発に減り、7〜17 m/s の弱い弾が増え、80 m/s の過速も 2 発)。採用しない。

残る課題: 20 発中 4 発が 38〜100 m/s の過速で ±22〜27 度へ飛ぶ。99.8 m/s は
射出輪の表面速度 32 m/s では出ないので、食い込みの貫入解消による力積。食い込みを
減らすと片輪だけの弾が増えるという相反があり、剛体のままでは詰めきれない。

Co-Authored-By: Claude Opus 5 (1M context) <noreply@anthropic.com>

File: colcon_ws/src/sample_robot_description/urdf/shooter/shooter.urdf.xacro (robot description, xacro)
@@ -9,14 +9,27 @@
     roller_squeeze     片側あたりの食い込み量。射出輪の間隔はこれで決まる:
                          y = ±(disc_radius + roller_radius - roller_squeeze)
-    roller_squeeze は 0.001 にしてある。以前は射出輪の中心が y = ±0.12、
-    半径 0.04 で内面が ±0.08、ディスク直径 0.18 に対して片側 10 mm も
-    食い込んでいた。剛体どうしでこれだけ貫入すると解消時に過大な力積が出て、
-    同じ指令でも足元に落ちる弾と 350 m 飛ぶ弾が混ざる。接線力で送り出すには
-    法線力が要るので 0 にはせず、わずかに噛ませる。
+    以前は射出輪の中心が y = ±0.12、半径 0.04 で内面が ±0.08、ディスク直径 0.18
+    に対して片側 10 mm も食い込んでいた。剛体どうしでこれだけ貫入すると解消時に
+    過大な力積が出て、同じ指令でも足元に落ちる弾と 350 m 飛ぶ弾が混ざる。接線力で
+    送り出すには法線力が要るので 0 にはせず、わずかに噛ませる。
+    wall_clearance  通路の壁とディスクの片側あたりの隙間。
+    食い込みは隙間より大きく取ること。小さいと、遊びの範囲でディスクが片側へ
+    寄ったとき反対側の輪に届かず、片輪だけで蹴られる。実測では射出の半数が
+    そうなっていて、正常な 33〜35 m/s に対して 10〜18 m/s しか出ず、方位も
+    -12〜+14 度に散っていた (両輪で噛んだ弾は +0.3〜+1.2 度に収まる)。
+    以前は隙間 10 mm に対して食い込み 1 mm だった。
   -->
   <xacro:property name="disc_radius"   value="0.09"/>
   <xacro:property name="roller_radius" value="0.04"/>
   <xacro:property name="roller_width"  value="0.03"/>
-  <xacro:property name="roller_squeeze" value="0.001"/>
+  <xacro:property name="roller_squeeze" value="0.002"/>
+  <xacro:property name="wall_thickness" value="0.02"/>
+  <xacro:property name="wall_clearance" value="0.0015"/>
+  <xacro:property name="wall_y"
+                  value="${disc_radius + wall_clearance + wall_thickness / 2}"/>
+  <!-- 通路は射出輪の前縁 (x = 0.15 - 0.04 = 0.11) まで案内する。以前は x = 0.10 で
+       終わっていて、噛む直前の 1 cm が無案内だった。 -->
+  <xacro:property name="wall_length" value="0.22"/>
+  <xacro:property name="wall_center_x" value="0.01"/>
   <xacro:property name="roller_offset"
                   value="${disc_radius + roller_radius - roller_squeeze}"/>
@@ -86,5 +99,5 @@
         </link>
         <joint name="shooter_wall1_link_joint" type="fixed">
-          <origin rpy="0 0 0" xyz="0.0 0.11 0.05"/>
+          <origin rpy="0 0 0" xyz="${wall_center_x} ${wall_y} 0.05"/>
           <parent link="shooter_base_link"/>
           <child link="shooter_wall1_link"/>
@@ -93,12 +106,12 @@
           <visual>
                 <geometry>
-                  <box size="0.2 0.02 0.08" />
-                </geometry>
-                <material name="shooter_unit"/>
-          </visual>
-          <collision>
-            <collision_material name="shooter_unit"/>
-                <geometry>
-                  <box size="0.2 0.02 0.08" />
+                  <box size="${wall_length} ${wall_thickness} 0.08" />
+                </geometry>
+                <material name="shooter_unit"/>
+          </visual>
+          <collision>
+            <collision_material name="shooter_unit"/>
+                <geometry>
+                  <box size="${wall_length} ${wall_thickness} 0.08" />
                 </geometry>
           </collision>
@@ -112,5 +125,5 @@
         </link>
         <joint name="shooter_wall2_link_joint" type="fixed">
-          <origin rpy="0 0 0" xyz="0.0 -0.11 0.05"/>
+          <origin rpy="0 0 0" xyz="${wall_center_x} ${-wall_y} 0.05"/>
           <parent link="shooter_base_link"/>
           <child link="shooter_wall2_link"/>
@@ -119,12 +132,12 @@
           <visual>
                 <geometry>
-                  <box size="0.2 0.02 0.08" />
-                </geometry>
-                <material name="shooter_unit"/>
-          </visual>
-          <collision>
-            <collision_material name="shooter_unit"/>
-                <geometry>
-                  <box size="0.2 0.02 0.08" />
+                  <box size="${wall_length} ${wall_thickness} 0.08" />
+                </geometry>
+                <material name="shooter_unit"/>
+          </visual>
+          <collision>
+            <collision_material name="shooter_unit"/>
+                <geometry>
+                  <box size="${wall_length} ${wall_thickness} 0.08" />
                 </geometry>
           </collision>

Commit message: [fix] 射出機構: 積み込み全体を壁で囲い、段の隙間を詰める
射出できない弾が 24% あった。原因を測って特定した。

射出直前の姿勢を 160 発ぶん記録し、射出の成否と突き合わせたところ、傾きが
決定的だった。

  傾き 0.00〜0.01 度   39/41 (95%)
  傾き 0.01〜0.02 度   40/40 (100%)
  傾き 0.02〜6.01 度   39/40 (98%)
  傾き 13.2〜89.9 度    4/39 (10%)

並べ替え検定でも成功群と失敗群の傾きの差は p = 0.000。高さのずれも同様に効く
(正規の z = 0.504 に座っていれば 100%、上下にずれると 36〜68%)。傾いた弾は
射出輪に噛まない。

なぜ傾くか。通路の壁は高さ 0.08 で、シュータ座標の z = 0.01〜0.09 しか囲えて
いなかった。ディスクは base_link 基準で z = 0.55 から 0.025 間隔に 20 枚積むので、
囲われているのは最下段の 1 枚だけ。上の 19 枚は横に支えの無い自立した積み重ねに
なっていて、崩れて傾く。

さらに間隔 0.025 はディスク厚 0.02 に対して 5 mm の隙間があり、各段が落下して
跳ねる。20 段ぶん積み上がると崩れる原因になる。

壁の高さを 0.585 にして積み込み全体を覆い、間隔を 0.021 (隙間 1 mm) にした。
壁の高さと中心はプロパティにしたので、枚数や間隔を変えるときはここも合わせる。

実測 (8 ラウンド x 20 発、姿勢を記録して射出の成否と対応付け):

  壁 0.08  / 間隔 0.025   射出 122/160 (76%)  傾き 6 度超 40 発 (25%)
  壁 0.585 / 間隔 0.025   射出 129/160 (81%)  傾き 6 度超 33 発 (21%)
  壁 0.585 / 間隔 0.021   射出 143/160 (89%)  傾き 6 度超 16 発 (10%)

Co-Authored-By: Claude Opus 5 (1M context) <noreply@anthropic.com>

File: colcon_ws/src/sample_robot_description/urdf/shooter/shooter.urdf.xacro (robot description, xacro)
@@ -33,4 +33,17 @@
   <xacro:property name="wall_center_x" value="0.01"/>
   <!--
+    壁の高さは積み込み全体を覆う。以前は 0.08 (シュータ座標で z = 0.01〜0.09) しか
+    なく、囲えていたのは最下段の 1 枚だけだった。ディスクは base_link 基準で
+    z = 0.55 から 0.025 間隔に 20 枚積むので、上の 19 枚は横に支えが無い自立した
+    積み重ねになり、崩れて傾く。
+    傾いた弾は射出輪に噛まない。実測 160 発で、傾き 6 度以下は 118/121 (98%) が
+    射出されたのに対し、13 度以上は 4/39 (10%) しか出ていない。射出失敗の 24% は
+    ここが原因だった。
+    積み込みの上端はシュータ座標で z = 0.575 なので、余裕を見て 0.595 まで覆う。
+    枚数や間隔を変えるときはここも合わせること。
+  -->
+  <xacro:property name="wall_height" value="0.585"/>
+  <xacro:property name="wall_center_z" value="${0.01 + wall_height / 2}"/>
+  <!--
     間隔には roller_contact_offset (common.xacro で定義) の増分も足す。
     contact_offset は接触を生成し始める距離なので、大きくすると触れる前から
@@ -107,5 +120,5 @@
         </link>
         <joint name="shooter_wall1_link_joint" type="fixed">
-          <origin rpy="0 0 0" xyz="${wall_center_x} ${wall_y} 0.05"/>
+          <origin rpy="0 0 0" xyz="${wall_center_x} ${wall_y} ${wall_center_z}"/>
           <parent link="shooter_base_link"/>
           <child link="shooter_wall1_link"/>
@@ -114,12 +127,12 @@
           <visual>
                 <geometry>
-                  <box size="${wall_length} ${wall_thickness} 0.08" />
-                </geometry>
-                <material name="shooter_unit"/>
-          </visual>
-          <collision>
-            <collision_material name="shooter_unit"/>
-                <geometry>
-                  <box size="${wall_length} ${wall_thickness} 0.08" />
+                  <box size="${wall_length} ${wall_thickness} ${wall_height}" />
+                </geometry>
+                <material name="shooter_unit"/>
+          </visual>
+          <collision>
+            <collision_material name="shooter_unit"/>
+                <geometry>
+                  <box size="${wall_length} ${wall_thickness} ${wall_height}" />
                 </geometry>
           </collision>
@@ -133,5 +146,5 @@
         </link>
         <joint name="shooter_wall2_link_joint" type="fixed">
-          <origin rpy="0 0 0" xyz="${wall_center_x} ${-wall_y} 0.05"/>
+          <origin rpy="0 0 0" xyz="${wall_center_x} ${-wall_y} ${wall_center_z}"/>
           <parent link="shooter_base_link"/>
           <child link="shooter_wall2_link"/>
@@ -140,12 +153,12 @@
           <visual>
                 <geometry>
-                  <box size="${wall_length} ${wall_thickness} 0.08" />
-                </geometry>
-                <material name="shooter_unit"/>
-          </visual>
-          <collision>
-            <collision_material name="shooter_unit"/>
-                <geometry>
-                  <box size="${wall_length} ${wall_thickness} 0.08" />
+                  <box size="${wall_length} ${wall_thickness} ${wall_height}" />
+                </geometry>
+                <material name="shooter_unit"/>
+          </visual>
+          <collision>
+            <collision_material name="shooter_unit"/>
+                <geometry>
+                  <box size="${wall_length} ${wall_thickness} ${wall_height}" />
                 </geometry>
           </collision>

Commit message: [change] ディスクを都度生成にし、射出を安定させる
起動時に 1 台 20 枚を積み上げるのをやめ、装填口に常に 1 枚だけ置く方式に
変える。積み荷は接触したまま積み重なった剛体でソルバのコストが高く、
2 台ぶんの 40 枚で物理が実時間に収まらなくなっていた (カメラ映像が
2.8 FPS まで低下)。同じ 40 枚でも撃ち終えて地面に散らばった状態なら
10.5 FPS 出る。静止した剛体はソルバから外れるため。

core_sim_utils/flying_disc_feeder を bring_up_core_stage から起動する。
装填口が空になったら 1 枚補充し、場のディスクは全機体あわせて 24 枚に保つ。
実測で 2 台構成で撃ち続けても RTF 1.000 / 10.00 FPS を維持する。

実装で踏んだ点:

- 生成は「引き戻しに転じた瞬間」ではなく「引き切ってから」。ストローク
  0.2 m を 1 m/s で戻るので 0.2 秒かかる一方、生成の往復は 100 ms しか
  ないため、転じた瞬間に置くとローダーがまだ通路の中にいて弾かれる。
  joint_states の位置を見て引き切りを待つ。
- 装填位置は機体の姿勢をそのまま使う (yaw だけでなく roll/pitch も)。
  フィールドの台に乗って持ち上がっても傾いても装填口が追従する。
  実測: 台 (上面 0.5 m) の上でも射出でき、機体を 8.2 度前上がりに
  傾けると射出仰角が +7.9 度になる (ほぼ 1:1 で追従)。
- 初速を付けた生成はできない。SpawnEntity に twist が無く、生成してから
  set_entity_state で与えると往復 2 回 (約 150 ms) の間に 11 cm 落ちる。
  射出輪の幅は 3 cm なので帯から外れる。底板に載せて装填機構で押す。
- 上限に達するまでは 1 枚も消さない。撃った端から消えると的に届かない。
  装填口に載っている弾も消さない。delete_entity は積み荷のディスクに
  対して応答が返らなくなった前例があるので、静止しているものだけを
  対象にし、打ち切り時間を設ける。

射出まわりも直す:

- バレル (押さえ) を通路の後端から射出輪の先まで伸ばす。以前は
  x +0.10〜+0.20 にしか無く、ディスクが待機する通路 (x -0.10〜+0.12) の
  上には何も無かった。
- teleop の射出輪速度を parameter 化し、既定を 800 から 500 rad/s
  (約 20 m/s) にする。実測 (各 3 回、10 ストロークずつ):
      250  実測  9.5 m/s  方位の幅 12 deg  破綻 0  射程 約 3 m
      500  実測 20.5 m/s  方位の幅 15 deg  破綻 0  射程 約 6 m
      800  実測 19.9 m/s  方位の幅 22 deg  破綻あり
  500 を超えても初速は伸びず、方位のばらつきと貫入由来の過速だけが増える。

measure_shoot.py は、試験中に現れたディスクを全部追跡するように直す。
開始時のスナップショットだけを見ていると、都度生成では名前が毎回変わるため
最初の 1 枚しか数えられない (28 ストロークで「0/1」と出たが、実際には
初速 30.8 m/s で正常に射出されていた)。

Co-Authored-By: Claude Opus 5 (1M context) <noreply@anthropic.com>

File: colcon_ws/src/sample_robot_description/urdf/shooter/shooter.urdf.xacro (robot description, xacro)
@@ -59,4 +59,25 @@
        反力を一切受け流さず、上の力積を増幅していた。800 rad/s での回転エネルギは
        この値でも 1 発 (7.7 J) に対して十分余裕がある。 -->
+  <!--
+    バレル (押さえ) の寸法。
+    ディスクは底板の上面 (シュータ座標 z = +0.04) に載り、厚み 0.02 なので
+    上面が +0.06。バレルの下面をそこから barrel_clearance だけ上に置くと、
+    通路で待っているディスクが浮き上がれなくなる。
+    以前はバレルが x +0.10〜+0.20 にしか無く、ディスクが待機する通路
+    (x -0.10〜+0.12) の上には何も無かった。押さえが無いぶん噛み方が安定せず、
+    初速がばらついていた (中央 25.8 m/s、理論 32 m/s)。通路の後端から
+    射出輪の先まで覆う長さに変える。
+  -->
+  <xacro:property name="barrel_clearance" value="0.005"/>
+  <xacro:property name="barrel_thickness" value="0.04"/>
+  <xacro:property name="barrel_back_x"  value="-0.12"/>
+  <xacro:property name="barrel_front_x" value="0.20"/>
+  <xacro:property name="barrel_length"
+                  value="${barrel_front_x - barrel_back_x}"/>
+  <xacro:property name="barrel_center_x"
+                  value="${(barrel_front_x + barrel_back_x) / 2}"/>
+  <!-- 下面 = ディスク上面 (0.06) + 隙間。中心はそこから厚みの半分だけ上。 -->
+  <xacro:property name="barrel_center_z"
+                  value="${0.06 + barrel_clearance + barrel_thickness / 2}"/>
   <xacro:property name="roller_mass"   value="0.5"/>
   <xacro:property name="roller_izz"
@@ -94,5 +115,5 @@
         </link>
         <joint name="shooter_barel_link_joint" type="fixed">
-          <origin rpy="0 0 0" xyz="0.15 0.0 0.09"/>
+          <origin rpy="0 0 0" xyz="${barrel_center_x} 0.0 ${barrel_center_z}"/>
           <parent link="shooter_base_link"/>
           <child link="shooter_barel_link"/>
@@ -101,12 +122,12 @@
           <visual>
                 <geometry>
-                  <box size="0.1 0.18 0.04" />
-                </geometry>
-                <material name="shooter_unit"/>
-          </visual>
-          <collision>
-            <collision_material name="shooter_unit"/>
-                <geometry>
-                  <box size="0.1 0.18 0.04" />
+                  <box size="${barrel_length} 0.18 ${barrel_thickness}" />
+                </geometry>
+                <material name="shooter_unit"/>
+          </visual>
+          <collision>
+            <collision_material name="shooter_unit"/>
+                <geometry>
+                  <box size="${barrel_length} 0.18 ${barrel_thickness}" />
                 </geometry>
           </collision>
