Commit message: [fix] 被弾判定: contact_count の増分で数えて取りこぼしを無くす
装甲板の被弾は Bool の立ち上がりを数えていたが、10 回に 1 回ほど取りこぼして
いた。原因は 2 つあった。

ひとつはセンサ側。ContactSensor は publish の瞬間に接触しているかしか見て
おらず、ディスクは物理 1〜数ステップ (5〜15 ms) しか触れないのに、publish は
描画フレームレートが上限で 100 ms 間隔しかない。サンプルの合間に始まって
終わった被弾は跡形も無く消えていた。update_rate を 30 Hz に書いても、
publisher が 1 フレームに 1 通しか出さないので実測 10 Hz のままで効かない。

もうひとつは経路。Unity から ros_tcp_endpoint への TCP は 1 本で、8 台ぶんの
カメラを積むと送信キューが溢れる。捨てられた通に立ち上がりが乗っていれば、
その被弾は永久に失われる。

シミュレータ側でラッチして数えるようにしたので (Unity_ROS2_Robot_Simulator
6506fd5)、累積値の差分を取る形に変えた。何通落ちても次の 1 通で追いつくし、
1 サンプルの間に 2 発当たった場合も差分は 2 になる。リセットや再スポーンで
カウンタが 0 に戻るため、値が減ったら被弾ではなく基準の取り直しとして扱う。

Bool とレンチは使わなくなったので URDF で止めた。装甲板 4 枚 x 8 機で毎秒
1920 通が経路から消える。update_rate は実際に出る 10 Hz に合わせた。

実測: 1 発ずつ 6 回と 10 発ずつ 2 回、計 8 試行でセンサの増分と HP の減少が
すべて一致した。機体に 4 回・7 回と跳ね返ったディスクでも増分は 1 と 0 で、
重複計上は出ていない。

Co-Authored-By: Claude Opus 5 (1M context) <noreply@anthropic.com>

File: colcon_ws/src/sample_robot_description/simulation/sample_robot.simulation.xacro (robot description, xacro)
@@ -8,6 +8,9 @@
     camera  -> /<robot>/<link>/image_raw   (sensor_msgs/Image)
                /<robot>/<link>/camera_info (sensor_msgs/CameraInfo)
-    contact -> /<robot>/<link>/contact         (std_msgs/Bool)
+    contact -> /<robot>/<link>/contact_count   (std_msgs/Int32)
+               /<robot>/<link>/contact         (std_msgs/Bool)
                /<robot>/<link>/contact/wrench  (geometry_msgs/WrenchStamped)
+  接触センサの後ろ 2 つは <publish_state> と <publish_wrench> を false に
+  すると止められます (既定は出す)。contact_count は常に出ます。
   Isaac 版はリンクの親子関係がトピック名に入り
   /<robot>/base_link/camera_link/image_raw でしたが、こちらはリンク名だけの
@@ -76,16 +79,38 @@
         </clip>
       </sensor>
-      <!-- 装甲板の被弾検出。hp_manager が std_msgs/Bool の立ち上がりを数える -->
+      <!--
+        装甲板の被弾検出。hp_manager が std_msgs/Int32 (contact_count) の
+        増分を数える。
+        Bool の立ち上がりではなくカウンタを使うのは、経路のどこで落ちても
+        次の 1 通で追いつけるため。Bool は落ちた通に立ち上がりが乗っていると
+        その被弾が永久に失われる。
+        update_rate はディスクの接触時間 (物理 1〜数ステップ) より必ず粗い。
+        それでも取りこぼさないのは、接触の到着をセンサ側で数えていて、
+        サンプルの合間に始まって終わった接触も残るため。ここが決めるのは
+        検出漏れではなく報告の遅れだけなので、描画フレームレートに合わせる。
+        publisher は 1 フレームに 1 通しか出さないので、これより上げても
+        通数は増えず、値が効かないまま実測 10 Hz になるだけ。
+        Bool とレンチは hp_manager が使わないので止める。装甲板 4 枚 x 8 機で
+        毎秒 960 通ずつ、合わせて 1920 通/秒が経路から消える。
+      -->
       <sensor name="armor1_link" type="contact">
-        <update_rate>30.0</update_rate>
+        <update_rate>10.0</update_rate>
+        <publish_state>false</publish_state>
+        <publish_wrench>false</publish_wrench>
       </sensor>
       <sensor name="armor2_link" type="contact">
-        <update_rate>30.0</update_rate>
+        <update_rate>10.0</update_rate>
+        <publish_state>false</publish_state>
+        <publish_wrench>false</publish_wrench>
       </sensor>
       <sensor name="armor3_link" type="contact">
-        <update_rate>30.0</update_rate>
+        <update_rate>10.0</update_rate>
+        <publish_state>false</publish_state>
+        <publish_wrench>false</publish_wrench>
       </sensor>
       <sensor name="armor4_link" type="contact">
-        <update_rate>30.0</update_rate>
+        <update_rate>10.0</update_rate>
+        <publish_state>false</publish_state>
+        <publish_wrench>false</publish_wrench>
       </sensor>
     </simulation>
