Commit message: [change] 走行をオムニホイールから車体への直接加力へ置き換える
オムニホイール 4 輪を外し、シミュレータ側の body_twist_drive
(/<機体名>/cmd_vel を直接購読して車体へ力を加える) で走らせる。

1 輪あたりフリーローラ 8 個 + ハウジング 2 個で、4 輪だと 40 リンクになり、
これが PhysX ソルバのコストの大半を占めていた。ロボット 2 台 + ディスク 40 枚で
物理が実時間に収まらなくなり、Unity が 1 フレームに maximumDeltaTime (既定
0.333 秒) ぶんの物理をまとめて回すため、カメラ映像が 2.8 FPS まで落ちていた。

実測 (physics_hz 200):

                          置き換え前   置き換え後
  2 台 + ディスク 40 枚    2.82 FPS     10.00 FPS
                          RTF 0.94     RTF 1.000
  8 台 (ディスクなし)      2.02 FPS      9.97 FPS
                          RTF 0.66     RTF 0.998
  前後・左右の指令追従        54%       99〜100%
  旋回の指令追従              82%      97〜100%
  1 台あたりのリンク数         69            29
  射出の装填成功率      57%/ストローク  100%/ストローク

速度を代入せず力で追従させているので、他機に押されるし押し返せる
(指令ゼロで静止している機体を 1.0 m/s で押して 2.82 m 動かせることを確認)。
移動しながらの射出も、前進・旋回・円運動のいずれでも成立する。

車輪を外すと車体が 5 cm 下がって床に直付きになり、フィールドの構造物に
引っ掛かって走れなくなる (上限の 156 N を掛けても速度 0)。車輪と同じ位置・
同じ半径の摩擦 0 の球を base_frame_link の collision として 4 個足して、
車高と地上高を戻している。リンクは増えない。車輪の見た目もハウジングの
STL を同じ位置に置いて残した (回転はしない)。

速度・加速度の上限は omni_wheel_controller の設定をそのまま
simulation/sample_robot.simulation.xacro へ移した。ただし以前は車輪が滑って
指令の 54% しか出ていなかったので、同じ指令でも実際の速度は約 1.85 倍になる。

ros2_control が担うのは射出機構だけになり、omni_wheel_controller と
velocity_pub は経路から外れた。odom は ground_truth で代替する。

この構成には Unity_ROS2_Robot_Simulator v1.1.0 以降が要るので、
docker/dockerfile の SIMULATOR_VERSION も上げてある。

Co-Authored-By: Claude Opus 5 (1M context) <noreply@anthropic.com>

File: colcon_ws/src/sample_robot_description/robots/sample_robot.urdf.xacro (robot description, xacro)
@@ -6,5 +6,4 @@
   <xacro:include filename="$(find sample_robot_description)/urdf/common.xacro"/>
   <xacro:include filename="$(find sample_robot_description)/urdf/base/base.urdf.xacro"/>
-  <xacro:include filename="$(find sample_robot_description)/urdf/wheel/wheel_100mm.urdf.xacro"/>
   <xacro:include filename="$(find sample_robot_description)/urdf/shooter/shooter.urdf.xacro"/>
   <xacro:include filename="$(find sample_robot_description)/simulation/sample_robot.simulation.xacro"/>
@@ -14,24 +13,14 @@
   <!-- Base -->
   <link name="base_link"/>
-  <xacro:base_v0 parent="base_link">
+  <xacro:base_v0 parent="base_link" skids="true">
 	<origin xyz="0 0 0.06"/>
   </xacro:base_v0>
-  <!-- Wheel -->
-  <!-- Wheel0 -->
-  <xacro:omni_wheel prefix="wheel0" parent="base_link">
-	  <origin xyz="0.35 0.35 0.05" rpy="0 ${pi/2} ${pi/4}"/>
-  </xacro:omni_wheel>
-  <!-- Wheel1 -->
-  <xacro:omni_wheel prefix="wheel1" parent="base_link">
-	  <origin xyz="-0.35 0.35 0.05" rpy="0 ${pi/2} ${pi*3/4}"/>
-  </xacro:omni_wheel>
-  <!-- Wheel3 -->
-  <xacro:omni_wheel prefix="wheel2" parent="base_link">
-	  <origin xyz="-0.35 -0.35 0.05" rpy="0 ${pi/2} ${-pi*3/4}"/>
-  </xacro:omni_wheel>
-  <!-- Wheel2 -->
-  <xacro:omni_wheel prefix="wheel3" parent="base_link">
-	  <origin xyz="0.35 -0.35 0.05" rpy="0 ${pi/2} ${-pi/4}"/>
-  </xacro:omni_wheel>
+  <!--
+    駆動系はここにあったオムニホイール 4 輪 (1 輪あたりフリーローラ 8 個 +
+    ハウジング 2 個、4 輪で 40 リンク) を外してある。走行はシミュレータ側の
+    body_twist_drive が車体へ直接力を加えて行う
+    (simulation/sample_robot.simulation.xacro を参照)。
+    接地と車輪の見た目は base_v0 の skids="true" が受け持つ。
+  -->
   <xacro:shooter_v0 parent="base_link">
 	<origin xyz="0 0 0.45"/>

File: colcon_ws/src/sample_robot_description/robots/sample_robot_1.urdf.xacro (robot description, xacro)
@@ -6,5 +6,4 @@
   <xacro:include filename="$(find sample_robot_description)/urdf/common.xacro"/>
   <xacro:include filename="$(find sample_robot_description)/urdf/base/base.urdf.xacro"/>
-  <xacro:include filename="$(find sample_robot_description)/urdf/wheel/wheel_100mm.urdf.xacro"/>
   <xacro:include filename="$(find sample_robot_description)/urdf/shooter/shooter.urdf.xacro"/>
   <xacro:include filename="$(find sample_robot_description)/simulation/sample_robot.simulation.xacro"/>
@@ -22,24 +21,14 @@
     </inertial>
   </link>
-  <xacro:base_v0 parent="base_link">
+  <xacro:base_v0 parent="base_link" skids="true">
 	<origin xyz="0 0 0.06"/>
   </xacro:base_v0>
-  <!-- Wheel -->
-  <!-- Wheel0 -->
-  <xacro:omni_wheel prefix="wheel0" parent="base_link">
-	  <origin xyz="0.35 0.35 0.05" rpy="0 ${pi/2} ${pi/4}"/>
-  </xacro:omni_wheel>
-  <!-- Wheel1 -->
-  <xacro:omni_wheel prefix="wheel1" parent="base_link">
-	  <origin xyz="-0.35 0.35 0.05" rpy="0 ${pi/2} ${pi*3/4}"/>
-  </xacro:omni_wheel>
-  <!-- Wheel3 -->
-  <xacro:omni_wheel prefix="wheel2" parent="base_link">
-	  <origin xyz="-0.35 -0.35 0.05" rpy="0 ${pi/2} ${-pi*3/4}"/>
-  </xacro:omni_wheel>
-  <!-- Wheel2 -->
-  <xacro:omni_wheel prefix="wheel3" parent="base_link">
-	  <origin xyz="0.35 -0.35 0.05" rpy="0 ${pi/2} ${-pi/4}"/>
-  </xacro:omni_wheel>
+  <!--
+    駆動系はここにあったオムニホイール 4 輪 (1 輪あたりフリーローラ 8 個 +
+    ハウジング 2 個、4 輪で 40 リンク) を外してある。走行はシミュレータ側の
+    body_twist_drive が車体へ直接力を加えて行う
+    (simulation/sample_robot.simulation.xacro を参照)。
+    接地と車輪の見た目は base_v0 の skids="true" が受け持つ。
+  -->
   <xacro:shooter_v0 parent="base_link">
 	<origin xyz="0 0 0.45"/>

File: colcon_ws/src/sample_robot_description/robots/sample_robot_2.urdf.xacro (robot description, xacro)
@@ -6,5 +6,4 @@
   <xacro:include filename="$(find sample_robot_description)/urdf/common.xacro"/>
   <xacro:include filename="$(find sample_robot_description)/urdf/base/base.urdf.xacro"/>
-  <xacro:include filename="$(find sample_robot_description)/urdf/wheel/wheel_100mm.urdf.xacro"/>
   <xacro:include filename="$(find sample_robot_description)/urdf/shooter/shooter.urdf.xacro"/>
   <xacro:include filename="$(find sample_robot_description)/simulation/sample_robot.simulation.xacro"/>
@@ -22,24 +21,14 @@
     </inertial>
   </link>
-  <xacro:base_v0 parent="base_link">
+  <xacro:base_v0 parent="base_link" skids="true">
 	<origin xyz="0 0 0.06"/>
   </xacro:base_v0>
-  <!-- Wheel -->
-  <!-- Wheel0 -->
-  <xacro:omni_wheel prefix="wheel0" parent="base_link">
-	  <origin xyz="0.35 0.35 0.05" rpy="0 ${pi/2} ${pi/4}"/>
-  </xacro:omni_wheel>
-  <!-- Wheel1 -->
-  <xacro:omni_wheel prefix="wheel1" parent="base_link">
-	  <origin xyz="-0.35 0.35 0.05" rpy="0 ${pi/2} ${pi*3/4}"/>
-  </xacro:omni_wheel>
-  <!-- Wheel3 -->
-  <xacro:omni_wheel prefix="wheel2" parent="base_link">
-	  <origin xyz="-0.35 -0.35 0.05" rpy="0 ${pi/2} ${-pi*3/4}"/>
-  </xacro:omni_wheel>
-  <!-- Wheel2 -->
-  <xacro:omni_wheel prefix="wheel3" parent="base_link">
-	  <origin xyz="0.35 -0.35 0.05" rpy="0 ${pi/2} ${-pi/4}"/>
-  </xacro:omni_wheel>
+  <!--
+    駆動系はここにあったオムニホイール 4 輪 (1 輪あたりフリーローラ 8 個 +
+    ハウジング 2 個、4 輪で 40 リンク) を外してある。走行はシミュレータ側の
+    body_twist_drive が車体へ直接力を加えて行う
+    (simulation/sample_robot.simulation.xacro を参照)。
+    接地と車輪の見た目は base_v0 の skids="true" が受け持つ。
+  -->
   <xacro:shooter_v0 parent="base_link">
 	<origin xyz="0 0 0.45"/>

File: colcon_ws/src/sample_robot_description/robots/sample_robot_3.urdf.xacro (robot description, xacro)
@@ -6,5 +6,4 @@
   <xacro:include filename="$(find sample_robot_description)/urdf/common.xacro"/>
   <xacro:include filename="$(find sample_robot_description)/urdf/base/base.urdf.xacro"/>
-  <xacro:include filename="$(find sample_robot_description)/urdf/wheel/wheel_100mm.urdf.xacro"/>
   <xacro:include filename="$(find sample_robot_description)/urdf/shooter/shooter.urdf.xacro"/>
   <xacro:include filename="$(find sample_robot_description)/simulation/sample_robot.simulation.xacro"/>
@@ -22,24 +21,14 @@
     </inertial>
   </link>
-  <xacro:base_v0 parent="base_link">
+  <xacro:base_v0 parent="base_link" skids="true">
 	<origin xyz="0 0 0.06"/>
   </xacro:base_v0>
-  <!-- Wheel -->
-  <!-- Wheel0 -->
-  <xacro:omni_wheel prefix="wheel0" parent="base_link">
-	  <origin xyz="0.35 0.35 0.05" rpy="0 ${pi/2} ${pi/4}"/>
-  </xacro:omni_wheel>
-  <!-- Wheel1 -->
-  <xacro:omni_wheel prefix="wheel1" parent="base_link">
-	  <origin xyz="-0.35 0.35 0.05" rpy="0 ${pi/2} ${pi*3/4}"/>
-  </xacro:omni_wheel>
-  <!-- Wheel3 -->
-  <xacro:omni_wheel prefix="wheel2" parent="base_link">
-	  <origin xyz="-0.35 -0.35 0.05" rpy="0 ${pi/2} ${-pi*3/4}"/>
-  </xacro:omni_wheel>
-  <!-- Wheel2 -->
-  <xacro:omni_wheel prefix="wheel3" parent="base_link">
-	  <origin xyz="0.35 -0.35 0.05" rpy="0 ${pi/2} ${-pi/4}"/>
-  </xacro:omni_wheel>
+  <!--
+    駆動系はここにあったオムニホイール 4 輪 (1 輪あたりフリーローラ 8 個 +
+    ハウジング 2 個、4 輪で 40 リンク) を外してある。走行はシミュレータ側の
+    body_twist_drive が車体へ直接力を加えて行う
+    (simulation/sample_robot.simulation.xacro を参照)。
+    接地と車輪の見た目は base_v0 の skids="true" が受け持つ。
+  -->
   <xacro:shooter_v0 parent="base_link">
 	<origin xyz="0 0 0.45"/>

File: colcon_ws/src/sample_robot_description/robots/sample_robot_4.urdf.xacro (robot description, xacro)
@@ -6,5 +6,4 @@
   <xacro:include filename="$(find sample_robot_description)/urdf/common.xacro"/>
   <xacro:include filename="$(find sample_robot_description)/urdf/base/base.urdf.xacro"/>
-  <xacro:include filename="$(find sample_robot_description)/urdf/wheel/wheel_100mm.urdf.xacro"/>
   <xacro:include filename="$(find sample_robot_description)/urdf/shooter/shooter.urdf.xacro"/>
   <xacro:include filename="$(find sample_robot_description)/simulation/sample_robot.simulation.xacro"/>
@@ -22,24 +21,14 @@
     </inertial>
   </link>
-  <xacro:base_v0 parent="base_link">
+  <xacro:base_v0 parent="base_link" skids="true">
 	<origin xyz="0 0 0.06"/>
   </xacro:base_v0>
-  <!-- Wheel -->
-  <!-- Wheel0 -->
-  <xacro:omni_wheel prefix="wheel0" parent="base_link">
-	  <origin xyz="0.35 0.35 0.05" rpy="0 ${pi/2} ${pi/4}"/>
-  </xacro:omni_wheel>
-  <!-- Wheel1 -->
-  <xacro:omni_wheel prefix="wheel1" parent="base_link">
-	  <origin xyz="-0.35 0.35 0.05" rpy="0 ${pi/2} ${pi*3/4}"/>
-  </xacro:omni_wheel>
-  <!-- Wheel3 -->
-  <xacro:omni_wheel prefix="wheel2" parent="base_link">
-	  <origin xyz="-0.35 -0.35 0.05" rpy="0 ${pi/2} ${-pi*3/4}"/>
-  </xacro:omni_wheel>
-  <!-- Wheel2 -->
-  <xacro:omni_wheel prefix="wheel3" parent="base_link">
-	  <origin xyz="0.35 -0.35 0.05" rpy="0 ${pi/2} ${-pi/4}"/>
-  </xacro:omni_wheel>
+  <!--
+    駆動系はここにあったオムニホイール 4 輪 (1 輪あたりフリーローラ 8 個 +
+    ハウジング 2 個、4 輪で 40 リンク) を外してある。走行はシミュレータ側の
+    body_twist_drive が車体へ直接力を加えて行う
+    (simulation/sample_robot.simulation.xacro を参照)。
+    接地と車輪の見た目は base_v0 の skids="true" が受け持つ。
+  -->
   <xacro:shooter_v0 parent="base_link">
 	<origin xyz="0 0 0.45"/>

File: colcon_ws/src/sample_robot_description/robots/sample_robot_5.urdf.xacro (robot description, xacro)
@@ -6,5 +6,4 @@
   <xacro:include filename="$(find sample_robot_description)/urdf/common.xacro"/>
   <xacro:include filename="$(find sample_robot_description)/urdf/base/base.urdf.xacro"/>
-  <xacro:include filename="$(find sample_robot_description)/urdf/wheel/wheel_100mm.urdf.xacro"/>
   <xacro:include filename="$(find sample_robot_description)/urdf/shooter/shooter.urdf.xacro"/>
   <xacro:include filename="$(find sample_robot_description)/simulation/sample_robot.simulation.xacro"/>
@@ -22,24 +21,14 @@
     </inertial>
   </link>
-  <xacro:base_v0 parent="base_link">
+  <xacro:base_v0 parent="base_link" skids="true">
 	<origin xyz="0 0 0.06"/>
   </xacro:base_v0>
-  <!-- Wheel -->
-  <!-- Wheel0 -->
-  <xacro:omni_wheel prefix="wheel0" parent="base_link">
-	  <origin xyz="0.35 0.35 0.05" rpy="0 ${pi/2} ${pi/4}"/>
-  </xacro:omni_wheel>
-  <!-- Wheel1 -->
-  <xacro:omni_wheel prefix="wheel1" parent="base_link">
-	  <origin xyz="-0.35 0.35 0.05" rpy="0 ${pi/2} ${pi*3/4}"/>
-  </xacro:omni_wheel>
-  <!-- Wheel3 -->
-  <xacro:omni_wheel prefix="wheel2" parent="base_link">
-	  <origin xyz="-0.35 -0.35 0.05" rpy="0 ${pi/2} ${-pi*3/4}"/>
-  </xacro:omni_wheel>
-  <!-- Wheel2 -->
-  <xacro:omni_wheel prefix="wheel3" parent="base_link">
-	  <origin xyz="0.35 -0.35 0.05" rpy="0 ${pi/2} ${-pi/4}"/>
-  </xacro:omni_wheel>
+  <!--
+    駆動系はここにあったオムニホイール 4 輪 (1 輪あたりフリーローラ 8 個 +
+    ハウジング 2 個、4 輪で 40 リンク) を外してある。走行はシミュレータ側の
+    body_twist_drive が車体へ直接力を加えて行う
+    (simulation/sample_robot.simulation.xacro を参照)。
+    接地と車輪の見た目は base_v0 の skids="true" が受け持つ。
+  -->
   <xacro:shooter_v0 parent="base_link">
 	<origin xyz="0 0 0.45"/>

File: colcon_ws/src/sample_robot_description/robots/sample_robot_6.urdf.xacro (robot description, xacro)
@@ -6,5 +6,4 @@
   <xacro:include filename="$(find sample_robot_description)/urdf/common.xacro"/>
   <xacro:include filename="$(find sample_robot_description)/urdf/base/base.urdf.xacro"/>
-  <xacro:include filename="$(find sample_robot_description)/urdf/wheel/wheel_100mm.urdf.xacro"/>
   <xacro:include filename="$(find sample_robot_description)/urdf/shooter/shooter.urdf.xacro"/>
   <xacro:include filename="$(find sample_robot_description)/simulation/sample_robot.simulation.xacro"/>
@@ -22,24 +21,14 @@
     </inertial>
   </link>
-  <xacro:base_v0 parent="base_link">
+  <xacro:base_v0 parent="base_link" skids="true">
 	<origin xyz="0 0 0.06"/>
   </xacro:base_v0>
-  <!-- Wheel -->
-  <!-- Wheel0 -->
-  <xacro:omni_wheel prefix="wheel0" parent="base_link">
-	  <origin xyz="0.35 0.35 0.05" rpy="0 ${pi/2} ${pi/4}"/>
-  </xacro:omni_wheel>
-  <!-- Wheel1 -->
-  <xacro:omni_wheel prefix="wheel1" parent="base_link">
-	  <origin xyz="-0.35 0.35 0.05" rpy="0 ${pi/2} ${pi*3/4}"/>
-  </xacro:omni_wheel>
-  <!-- Wheel3 -->
-  <xacro:omni_wheel prefix="wheel2" parent="base_link">
-	  <origin xyz="-0.35 -0.35 0.05" rpy="0 ${pi/2} ${-pi*3/4}"/>
-  </xacro:omni_wheel>
-  <!-- Wheel2 -->
-  <xacro:omni_wheel prefix="wheel3" parent="base_link">
-	  <origin xyz="0.35 -0.35 0.05" rpy="0 ${pi/2} ${-pi/4}"/>
-  </xacro:omni_wheel>
+  <!--
+    駆動系はここにあったオムニホイール 4 輪 (1 輪あたりフリーローラ 8 個 +
+    ハウジング 2 個、4 輪で 40 リンク) を外してある。走行はシミュレータ側の
+    body_twist_drive が車体へ直接力を加えて行う
+    (simulation/sample_robot.simulation.xacro を参照)。
+    接地と車輪の見た目は base_v0 の skids="true" が受け持つ。
+  -->
   <xacro:shooter_v0 parent="base_link">
 	<origin xyz="0 0 0.45"/>

File: colcon_ws/src/sample_robot_description/robots/sample_robot_7.urdf.xacro (robot description, xacro)
@@ -6,5 +6,4 @@
   <xacro:include filename="$(find sample_robot_description)/urdf/common.xacro"/>
   <xacro:include filename="$(find sample_robot_description)/urdf/base/base.urdf.xacro"/>
-  <xacro:include filename="$(find sample_robot_description)/urdf/wheel/wheel_100mm.urdf.xacro"/>
   <xacro:include filename="$(find sample_robot_description)/urdf/shooter/shooter.urdf.xacro"/>
   <xacro:include filename="$(find sample_robot_description)/simulation/sample_robot.simulation.xacro"/>
@@ -22,24 +21,14 @@
     </inertial>
   </link>
-  <xacro:base_v0 parent="base_link">
+  <xacro:base_v0 parent="base_link" skids="true">
 	<origin xyz="0 0 0.06"/>
   </xacro:base_v0>
-  <!-- Wheel -->
-  <!-- Wheel0 -->
-  <xacro:omni_wheel prefix="wheel0" parent="base_link">
-	  <origin xyz="0.35 0.35 0.05" rpy="0 ${pi/2} ${pi/4}"/>
-  </xacro:omni_wheel>
-  <!-- Wheel1 -->
-  <xacro:omni_wheel prefix="wheel1" parent="base_link">
-	  <origin xyz="-0.35 0.35 0.05" rpy="0 ${pi/2} ${pi*3/4}"/>
-  </xacro:omni_wheel>
-  <!-- Wheel3 -->
-  <xacro:omni_wheel prefix="wheel2" parent="base_link">
-	  <origin xyz="-0.35 -0.35 0.05" rpy="0 ${pi/2} ${-pi*3/4}"/>
-  </xacro:omni_wheel>
-  <!-- Wheel2 -->
-  <xacro:omni_wheel prefix="wheel3" parent="base_link">
-	  <origin xyz="0.35 -0.35 0.05" rpy="0 ${pi/2} ${-pi/4}"/>
-  </xacro:omni_wheel>
+  <!--
+    駆動系はここにあったオムニホイール 4 輪 (1 輪あたりフリーローラ 8 個 +
+    ハウジング 2 個、4 輪で 40 リンク) を外してある。走行はシミュレータ側の
+    body_twist_drive が車体へ直接力を加えて行う
+    (simulation/sample_robot.simulation.xacro を参照)。
+    接地と車輪の見た目は base_v0 の skids="true" が受け持つ。
+  -->
   <xacro:shooter_v0 parent="base_link">
 	<origin xyz="0 0 0.45"/>

File: colcon_ws/src/sample_robot_description/robots/sample_robot_8.urdf.xacro (robot description, xacro)
@@ -6,5 +6,4 @@
   <xacro:include filename="$(find sample_robot_description)/urdf/common.xacro"/>
   <xacro:include filename="$(find sample_robot_description)/urdf/base/base.urdf.xacro"/>
-  <xacro:include filename="$(find sample_robot_description)/urdf/wheel/wheel_100mm.urdf.xacro"/>
   <xacro:include filename="$(find sample_robot_description)/urdf/shooter/shooter.urdf.xacro"/>
   <xacro:include filename="$(find sample_robot_description)/simulation/sample_robot.simulation.xacro"/>
@@ -22,24 +21,14 @@
     </inertial>
   </link>
-  <xacro:base_v0 parent="base_link">
+  <xacro:base_v0 parent="base_link" skids="true">
 	<origin xyz="0 0 0.06"/>
   </xacro:base_v0>
-  <!-- Wheel -->
-  <!-- Wheel0 -->
-  <xacro:omni_wheel prefix="wheel0" parent="base_link">
-	  <origin xyz="0.35 0.35 0.05" rpy="0 ${pi/2} ${pi/4}"/>
-  </xacro:omni_wheel>
-  <!-- Wheel1 -->
-  <xacro:omni_wheel prefix="wheel1" parent="base_link">
-	  <origin xyz="-0.35 0.35 0.05" rpy="0 ${pi/2} ${pi*3/4}"/>
-  </xacro:omni_wheel>
-  <!-- Wheel3 -->
-  <xacro:omni_wheel prefix="wheel2" parent="base_link">
-	  <origin xyz="-0.35 -0.35 0.05" rpy="0 ${pi/2} ${-pi*3/4}"/>
-  </xacro:omni_wheel>
-  <!-- Wheel2 -->
-  <xacro:omni_wheel prefix="wheel3" parent="base_link">
-	  <origin xyz="0.35 -0.35 0.05" rpy="0 ${pi/2} ${-pi/4}"/>
-  </xacro:omni_wheel>
+  <!--
+    駆動系はここにあったオムニホイール 4 輪 (1 輪あたりフリーローラ 8 個 +
+    ハウジング 2 個、4 輪で 40 リンク) を外してある。走行はシミュレータ側の
+    body_twist_drive が車体へ直接力を加えて行う
+    (simulation/sample_robot.simulation.xacro を参照)。
+    接地と車輪の見た目は base_v0 の skids="true" が受け持つ。
+  -->
   <xacro:shooter_v0 parent="base_link">
 	<origin xyz="0 0 0.45"/>

File: colcon_ws/src/sample_robot_description/ros2_control/sample_robot.ros2_control.xacro (robot description, xacro)
@@ -2,4 +2,9 @@
 <robot xmlns:xacro="http://www.ros.org/wiki/xacro">
   <xacro:macro name="sample_robot_ros2_control" params="name use_fake_hardware:=^|false fake_sensor_commands:=^|false use_sim:=^|false">
+    <!--
+      ros2_control が担うのは射出機構だけ。走行はシミュレータ側の
+      body_twist_drive (simulation/sample_robot.simulation.xacro) が
+      /<機体名>/cmd_vel を直接受け取って行うので、車輪の関節は無くなった。
+    -->
     <ros2_control name="${name}" type="system">
       <hardware>
@@ -34,48 +39,4 @@
         </xacro:if>
       </hardware>
-      <joint name="wheel0_shaft_joint">
-        <command_interface name="velocity">
-          <param name="min">-100</param>
-          <param name="max">100</param>
-        </command_interface>
-        <state_interface name="position">
-          <param name="initial_value">0.0</param>
-        </state_interface>
-        <state_interface name="velocity"/>
-        <state_interface name="effort"/>
-      </joint>
-      <joint name="wheel1_shaft_joint">
-        <command_interface name="velocity">
-          <param name="min">-100</param>
-          <param name="max">100</param>
-        </command_interface>
-        <state_interface name="position">
-          <param name="initial_value">0.0</param>
-        </state_interface>
-        <state_interface name="velocity"/>
-        <state_interface name="effort"/>
-      </joint>
-      <joint name="wheel2_shaft_joint">
-        <command_interface name="velocity">
-          <param name="min">-100</param>
-          <param name="max">100</param>
-        </command_interface>
-        <state_interface name="position">
-          <param name="initial_value">0.0</param>
-        </state_interface>
-        <state_interface name="velocity"/>
-        <state_interface name="effort"/>
-      </joint>
-      <joint name="wheel3_shaft_joint">
-        <command_interface name="velocity">
-          <param name="min">-100</param>
-          <param name="max">100</param>
-        </command_interface>
-        <state_interface name="position">
-          <param name="initial_value">0.0</param>
-        </state_interface>
-        <state_interface name="velocity"/>
-        <state_interface name="effort"/>
-      </joint>
       <joint name="shooter_wheel1_link_joint">
         <command_interface name="velocity">

File: colcon_ws/src/sample_robot_description/simulation/sample_robot.simulation.xacro (robot description, xacro)
@@ -18,4 +18,36 @@
     <!-- =============== Unity Simulator =============== -->
     <simulation>
+      <!--
+        車体速度による駆動。/<エンティティ名>/cmd_vel (geometry_msgs/Twist) を
+        シミュレータが直接購読し、各物理ステップで「指令速度 - 現在速度」を
+        詰めるのに要る力・トルクを車体へ加える。
+        オムニホイールの置き換え。フリーローラ 8 個 x 4 輪 + ハウジングで
+        1 台あたり 40 リンクあり、これがソルバのコストの大半を占めていた。
+        置き換えで 8 台同時でも RTF 1.0 / 10 FPS が出る (置き換え前は
+        RTF 0.66 / 2.0 FPS)。指令への追従も 54% から 100% になる。
+        速度代入ではなく加力なので、他機に押されるし、押し返せる。
+        上限値は置き換え前の omni_wheel_controller の設定をそのまま引き継ぐ
+        (linear.x: max_velocity 1.0 / max_acceleration 0.4、
+         angular.z: max_velocity 1.5 / max_acceleration 0.8)。
+        ただし以前は車輪が滑って指令の 54% しか出ていなかったので、
+        同じ指令でも実際の速度は約 1.85 倍になる。競技の間合いが変わるため、
+        必要なら max_linear_velocity を 0.54 前後まで落として合わせること。
+        command_timeout は omni_wheel_controller の cmd_vel_timeout に相当する。
+        指令が途切れた機体が走り続けないようにするためのもの。接地脚は
+        摩擦 0 なので、これが無いと止まらない。
+      -->
+      <!--
+        command_topic は書かないこと。書くと entity_namespace (spawn_entity は
+        空で投げる) がそのまま使われ、8 台全部が 1 本の /cmd_vel を共有して
+        一斉に同じ指令で動く。省略すればセンサと同じ /<エンティティ名>/cmd_vel
+        になり、機体ごとに分かれる。
+      -->
+      <sensor name="base_frame_link" type="body_twist_drive">
+        <max_linear_velocity>1.0</max_linear_velocity>
+        <max_angular_velocity>1.5</max_angular_velocity>
+        <max_linear_acceleration>0.4</max_linear_acceleration>
+        <max_angular_acceleration>0.8</max_angular_acceleration>
+        <command_timeout>0.5</command_timeout>
+      </sensor>
       <!-- 操縦用の一人称カメラ (720p) -->
       <sensor name="camera_link" type="camera">
