Commit message: [change] 走行をオムニホイールから車体への直接加力へ置き換える
オムニホイール 4 輪を外し、シミュレータ側の body_twist_drive
(/<機体名>/cmd_vel を直接購読して車体へ力を加える) で走らせる。

1 輪あたりフリーローラ 8 個 + ハウジング 2 個で、4 輪だと 40 リンクになり、
これが PhysX ソルバのコストの大半を占めていた。ロボット 2 台 + ディスク 40 枚で
物理が実時間に収まらなくなり、Unity が 1 フレームに maximumDeltaTime (既定
0.333 秒) ぶんの物理をまとめて回すため、カメラ映像が 2.8 FPS まで落ちていた。

実測 (physics_hz 200):

                          置き換え前   置き換え後
  2 台 + ディスク 40 枚    2.82 FPS     10.00 FPS
                          RTF 0.94     RTF 1.000
  8 台 (ディスクなし)      2.02 FPS      9.97 FPS
                          RTF 0.66     RTF 0.998
  前後・左右の指令追従        54%       99〜100%
  旋回の指令追従              82%      97〜100%
  1 台あたりのリンク数         69            29
  射出の装填成功率      57%/ストローク  100%/ストローク

速度を代入せず力で追従させているので、他機に押されるし押し返せる
(指令ゼロで静止している機体を 1.0 m/s で押して 2.82 m 動かせることを確認)。
移動しながらの射出も、前進・旋回・円運動のいずれでも成立する。

車輪を外すと車体が 5 cm 下がって床に直付きになり、フィールドの構造物に
引っ掛かって走れなくなる (上限の 156 N を掛けても速度 0)。車輪と同じ位置・
同じ半径の摩擦 0 の球を base_frame_link の collision として 4 個足して、
車高と地上高を戻している。リンクは増えない。車輪の見た目もハウジングの
STL を同じ位置に置いて残した (回転はしない)。

速度・加速度の上限は omni_wheel_controller の設定をそのまま
simulation/sample_robot.simulation.xacro へ移した。ただし以前は車輪が滑って
指令の 54% しか出ていなかったので、同じ指令でも実際の速度は約 1.85 倍になる。

ros2_control が担うのは射出機構だけになり、omni_wheel_controller と
velocity_pub は経路から外れた。odom は ground_truth で代替する。

この構成には Unity_ROS2_Robot_Simulator v1.1.0 以降が要るので、
docker/dockerfile の SIMULATOR_VERSION も上げてある。

Co-Authored-By: Claude Opus 5 (1M context) <noreply@anthropic.com>

File: colcon_ws/src/sample_robot_description/urdf/base/base.urdf.xacro (robot description, xacro)
@@ -2,5 +2,37 @@
 <robot xmlns:xacro="http://ros.org/wiki/xacro">
   <xacro:include filename="$(find sample_robot_description)/urdf/base/base.gazebo.xacro"/>
-  <xacro:macro name="base_v0" params="parent *joint_origin">
+  <!--
+    接地脚 1 個ぶん。車体を床から浮かせる球の当たり判定と、車輪の見た目を
+    base_frame_link へ直に足す。リンクもジョイントも増やさないので、
+    ソルバのコストは変わらない。
+    位置はオムニホイールの取り付け位置 (base_link 基準で ±0.35, ±0.35, 0.05)
+    に合わせる。base_frame_link は base_link の +0.06 なので z は -0.01。
+    半径 0.05 は車輪半径と同じで、これで車体下面の地上高 5 cm が元どおりになる。
+    車輪を外すと車体が 5 cm 下がって床に直付きになり、フィールドの構造物に
+    引っ掛かって走れなくなる (実測: 脚なしでは 156 N を掛けても速度 0、
+    脚ありで指令の 100%)。見た目もハウジングの STL をそのまま置いて、
+    車輪があるように見せる (回転はしない)。
+  -->
+  <xacro:macro name="base_skid" params="x y yaw">
+        <visual>
+          <origin xyz="${x} ${y} -0.01" rpy="0 ${pi/2} ${yaw}"/>
+          <geometry>
+            <mesh filename="file://$(find sample_robot_description)/meshes/STL/omni_housing_100mm.stl" />
+          </geometry>
+          <material name="gray"/>
+        </visual>
+        <collision>
+          <collision_material name="skid"/>
+          <origin xyz="${x} ${y} -0.01"/>
+          <geometry>
+            <sphere radius="0.05"/>
+          </geometry>
+        </collision>
+  </xacro:macro>
+  <!--
+    skids:=true で接地脚を付ける。BodyTwistDrive で走らせる構成用。
+    オムニホイールを付ける構成では false のままにすること (二重に接地する)。
+  -->
+  <xacro:macro name="base_v0" params="parent *joint_origin skids:=false">
         <joint name="base_frame_link_joint" type="fixed">
           <xacro:insert_block name="joint_origin"/>
@@ -21,4 +53,10 @@
                 </geometry>
           </collision>
+          <xacro:if value="${skids}">
+            <xacro:base_skid x="0.35"  y="0.35"  yaw="${pi/4}"/>
+            <xacro:base_skid x="-0.35" y="0.35"  yaw="${pi*3/4}"/>
+            <xacro:base_skid x="-0.35" y="-0.35" yaw="${-pi*3/4}"/>
+            <xacro:base_skid x="0.35"  y="-0.35" yaw="${-pi/4}"/>
+          </xacro:if>
           <inertial>
                 <origin xyz="0 0 0"/>

File: colcon_ws/src/sample_robot_description/urdf/common.xacro (robot description, xacro)
@@ -18,4 +18,13 @@
     <collision_material name="wheel_barrel">
       <friction static="1.0" dynamic="1.0" combine="maximum"/>
+    </collision_material>
+    <!--
+      接地脚。オムニホイールを BodyTwistDrive (車体への直接加力) へ置き換えた
+      構成で、車体を床から浮かせるためだけに使う球。推進は加力で行うので、
+      床とは擦らせない。combine="minimum" は床の材質 (Unity 既定 0.6) に
+      関わらず 0 を効かせるため。
+    -->
+    <collision_material name="skid">
+      <friction static="0.0" dynamic="0.0" combine="minimum"/>
     </collision_material>
     <!-- 車体・バンパ・装甲 -->

Commit message: [change] 射出口を下げて仰角 3.4 度を付ける
装甲板の帯 (base_link の 0.375〜0.525) に弾道ができるだけ長く留まるように、
射出口の高さと仰角を決め直す。従来は射出口 0.505・仰角 0 で、弾は撃った直後
から落ちるだけだった。

装甲板の高さの半分 (0.075 m) に収まる条件で初速 20 m/s の放物線を最適化すると
射出口 0.415 m・仰角 3.4 度になる。帯に留まる距離は 3.26 m から 4.87 m。
仰角を浅く取ってあるのは射出のばらつきに対する余裕を残すため。深い仰角ほど
帯の端をなぞるので、ばらつきで一気に外れる。

実測 (20 ストロークで装甲板のセンサが立ち上がった回数):

           変更前   変更後
    2 m      --      13 回
    3 m      10 回    9 回
    4 m       2 回    5 回

弾道も設計どおりで、射出口 0.409 m (設計 0.415)、仰角の中央値 +1.8〜+2.7 度、
前方 2 m まで帯に留まる。仰角のばらつきも幅 6.2 度から 4.4 度へ縮んだ
(射出口を下げて通路とバレルの拘束が効いた可能性があるが未確認)。

取り付け高さは射出口の目標高さから逆算する。仰角を付けると射出輪の位置が
回るので、その分を差し引かないと狙った高さにならない。
shooter_muzzle_z と shooter_elevation を変えれば取り付けは追従する。

装填口の高さもシュータに合わせて 0.50 から 0.4011 へ下げる。ここがずれると
通路に入らずバレルの上に乗って 1 発も射出できなくなる。

Co-Authored-By: Claude Opus 5 (1M context) <noreply@anthropic.com>

File: colcon_ws/src/sample_robot_description/robots/sample_robot.urdf.xacro (robot description, xacro)
@@ -23,6 +23,7 @@
     接地と車輪の見た目は base_v0 の skids="true" が受け持つ。
   -->
+  <!-- 取り付け高さと仰角は shooter.urdf.xacro で射出口の目標高さから逆算する -->
   <xacro:shooter_v0 parent="base_link">
-	<origin xyz="0 0 0.45"/>
+	<origin xyz="0 0 ${shooter_mount_z}" rpy="0 ${-shooter_elevation} 0"/>
   </xacro:shooter_v0>
   <!-- Base -->

File: colcon_ws/src/sample_robot_description/robots/sample_robot_1.urdf.xacro (robot description, xacro)
@@ -31,6 +31,7 @@
     接地と車輪の見た目は base_v0 の skids="true" が受け持つ。
   -->
+  <!-- 取り付け高さと仰角は shooter.urdf.xacro で射出口の目標高さから逆算する -->
   <xacro:shooter_v0 parent="base_link">
-	<origin xyz="0 0 0.45"/>
+	<origin xyz="0 0 ${shooter_mount_z}" rpy="0 ${-shooter_elevation} 0"/>
   </xacro:shooter_v0>
   <!-- Base -->

File: colcon_ws/src/sample_robot_description/robots/sample_robot_2.urdf.xacro (robot description, xacro)
@@ -31,6 +31,7 @@
     接地と車輪の見た目は base_v0 の skids="true" が受け持つ。
   -->
+  <!-- 取り付け高さと仰角は shooter.urdf.xacro で射出口の目標高さから逆算する -->
   <xacro:shooter_v0 parent="base_link">
-	<origin xyz="0 0 0.45"/>
+	<origin xyz="0 0 ${shooter_mount_z}" rpy="0 ${-shooter_elevation} 0"/>
   </xacro:shooter_v0>
   <!-- Base -->

File: colcon_ws/src/sample_robot_description/robots/sample_robot_3.urdf.xacro (robot description, xacro)
@@ -31,6 +31,7 @@
     接地と車輪の見た目は base_v0 の skids="true" が受け持つ。
   -->
+  <!-- 取り付け高さと仰角は shooter.urdf.xacro で射出口の目標高さから逆算する -->
   <xacro:shooter_v0 parent="base_link">
-	<origin xyz="0 0 0.45"/>
+	<origin xyz="0 0 ${shooter_mount_z}" rpy="0 ${-shooter_elevation} 0"/>
   </xacro:shooter_v0>
   <!-- Base -->

File: colcon_ws/src/sample_robot_description/robots/sample_robot_4.urdf.xacro (robot description, xacro)
@@ -31,6 +31,7 @@
     接地と車輪の見た目は base_v0 の skids="true" が受け持つ。
   -->
+  <!-- 取り付け高さと仰角は shooter.urdf.xacro で射出口の目標高さから逆算する -->
   <xacro:shooter_v0 parent="base_link">
-	<origin xyz="0 0 0.45"/>
+	<origin xyz="0 0 ${shooter_mount_z}" rpy="0 ${-shooter_elevation} 0"/>
   </xacro:shooter_v0>
   <!-- Base -->

File: colcon_ws/src/sample_robot_description/robots/sample_robot_5.urdf.xacro (robot description, xacro)
@@ -31,6 +31,7 @@
     接地と車輪の見た目は base_v0 の skids="true" が受け持つ。
   -->
+  <!-- 取り付け高さと仰角は shooter.urdf.xacro で射出口の目標高さから逆算する -->
   <xacro:shooter_v0 parent="base_link">
-	<origin xyz="0 0 0.45"/>
+	<origin xyz="0 0 ${shooter_mount_z}" rpy="0 ${-shooter_elevation} 0"/>
   </xacro:shooter_v0>
   <!-- Base -->

File: colcon_ws/src/sample_robot_description/robots/sample_robot_6.urdf.xacro (robot description, xacro)
@@ -31,6 +31,7 @@
     接地と車輪の見た目は base_v0 の skids="true" が受け持つ。
   -->
+  <!-- 取り付け高さと仰角は shooter.urdf.xacro で射出口の目標高さから逆算する -->
   <xacro:shooter_v0 parent="base_link">
-	<origin xyz="0 0 0.45"/>
+	<origin xyz="0 0 ${shooter_mount_z}" rpy="0 ${-shooter_elevation} 0"/>
   </xacro:shooter_v0>
   <!-- Base -->

File: colcon_ws/src/sample_robot_description/robots/sample_robot_7.urdf.xacro (robot description, xacro)
@@ -31,6 +31,7 @@
     接地と車輪の見た目は base_v0 の skids="true" が受け持つ。
   -->
+  <!-- 取り付け高さと仰角は shooter.urdf.xacro で射出口の目標高さから逆算する -->
   <xacro:shooter_v0 parent="base_link">
-	<origin xyz="0 0 0.45"/>
+	<origin xyz="0 0 ${shooter_mount_z}" rpy="0 ${-shooter_elevation} 0"/>
   </xacro:shooter_v0>
   <!-- Base -->

File: colcon_ws/src/sample_robot_description/robots/sample_robot_8.urdf.xacro (robot description, xacro)
@@ -31,6 +31,7 @@
     接地と車輪の見た目は base_v0 の skids="true" が受け持つ。
   -->
+  <!-- 取り付け高さと仰角は shooter.urdf.xacro で射出口の目標高さから逆算する -->
   <xacro:shooter_v0 parent="base_link">
-	<origin xyz="0 0 0.45"/>
+	<origin xyz="0 0 ${shooter_mount_z}" rpy="0 ${-shooter_elevation} 0"/>
   </xacro:shooter_v0>
   <!-- Base -->

File: colcon_ws/src/sample_robot_description/urdf/shooter/shooter.urdf.xacro (robot description, xacro)
@@ -69,4 +69,24 @@
     射出輪の先まで覆う長さに変える。
   -->
+  <!--
+    射出口の高さと仰角。装甲板の帯 (base_link の 0.375〜0.525) に弾道が
+    できるだけ長く留まるように決めた値。
+    装甲板の高さの半分 (0.075 m、中心 0.45 の上下 0.0375) に収まる条件で
+    初速 20 m/s の放物線を最適化すると、射出口 0.415 m・仰角 3.4 度で
+    帯に 4.87 m 留まる (仰角 0・射出口 0.505 の従来は 3.26 m)。
+    仰角を浅く取ってあるのは、射出のばらつきに対する余裕を残すため。
+    実測の仰角の幅は 6 度前後あり、±2 度ずれると装甲板全体で 1.43 m しか
+    保証できない。帯の端をなぞる深い仰角にすると、ばらつきでさらに短くなる。
+    取り付け高さは射出口の目標高さから逆算する。仰角を付けると射出輪の
+    位置が回るので、その分を差し引かないと狙った高さにならない。
+  -->
+  <xacro:property name="shooter_elevation" value="${radians(3.4)}"/>
+  <xacro:property name="shooter_muzzle_z" value="0.415"/>
+  <xacro:property name="roller_mount_x" value="0.15"/>
+  <xacro:property name="roller_mount_z" value="0.055"/>
+  <xacro:property name="shooter_mount_z"
+                  value="${shooter_muzzle_z
+                          - (roller_mount_x * sin(shooter_elevation)
+                             + roller_mount_z * cos(shooter_elevation))}"/>
   <xacro:property name="barrel_clearance" value="0.005"/>
   <xacro:property name="barrel_thickness" value="0.04"/>
@@ -493,5 +513,5 @@
         </link>
          <joint name="shooter_wheel1_link_joint" type="continuous">
-          <origin rpy="0 0 0" xyz="0.15 ${roller_offset} 0.055"/>
+          <origin rpy="0 0 0" xyz="${roller_mount_x} ${roller_offset} ${roller_mount_z}"/>
           <parent link="shooter_base_link"/>
           <child link="shooter_wheel1_link"/>
@@ -525,5 +545,5 @@
         </link>
          <joint name="shooter_wheel2_link_joint" type="continuous">
-          <origin rpy="0 0 0" xyz="0.15 ${-roller_offset} 0.055"/>
+          <origin rpy="0 0 0" xyz="${roller_mount_x} ${-roller_offset} ${roller_mount_z}"/>
           <parent link="shooter_base_link"/>
           <child link="shooter_wheel2_link"/>

Commit message: [fix] カメラを JPEG で受け取り、8 機すべてを 10 FPS に揃える
960x540 の生画像でも 8 機ぶん (一人称と俯瞰で 16 本) を流すと、Unity から
ros_tcp_endpoint への 1 本の TCP が溢れて 20 秒に 16251 通が捨てられていた。
捨てられ方は 1 フレーム内の publish 順に効くので、番号の大きい機体ほど映像が
落ちる。8 号機は 8.80 FPS で、1 号機との差が残っていた。

シミュレータ側で JPEG に符号化してから渡す (Unity_ROS2_Robot_Simulator
67f5171)。符号化はワーカースレッドで走るため物理演算とは競合しない。

  jpeg  全機 10.10 FPS  廃棄    23 件
  raw   8.80〜10.45     廃棄 16251 件

FPS も廃棄も jpeg が上回るので既定にする。生画像が要る用途のために
CORE_CAMERA_FORMAT=raw で戻せるようにしてあるが、launch 引数ではなく環境変数
なのは、URDF を組み立てる xacro が launch の実行前に走るため。置換オブジェクト
のままでは xacro に渡せない。

publisher_node は input_format で購読する型を選ぶ。復号は to_bgr に寄せた。

capture_image_topic.py も CompressedImage を受けられるようにした。既定が jpeg
になると image_raw が出なくなり、このスクリプトが一人称カメラを撮れなくなる。

Co-Authored-By: Claude Opus 5 (1M context) <noreply@anthropic.com>

File: colcon_ws/src/sample_robot_description/robots/sample_robot.urdf.xacro (robot description, xacro)
@@ -3,4 +3,6 @@
   <xacro:arg name="prefix" default="" />
   <xacro:arg name="use_sim" default="false" />
+  <!-- raw か jpeg。台数を積む構成では jpeg で経路の詰まりを避ける -->
+  <xacro:arg name="camera_format" default="raw" />
   <xacro:arg name="robot_name" default="sample_robot"/>
   <xacro:include filename="$(find sample_robot_description)/urdf/common.xacro"/>
@@ -140,5 +142,5 @@
     </inertial>
   </link>
-  <xacro:sample_robot_simulation prefix=""/>
+  <xacro:sample_robot_simulation prefix="" camera_format="$(arg camera_format)"/>
   <xacro:sample_robot_ros2_control name="$(arg robot_name)" use_sim="$(arg use_sim)"/>
 </robot>

File: colcon_ws/src/sample_robot_description/robots/sample_robot_1.urdf.xacro (robot description, xacro)
@@ -3,4 +3,6 @@
   <xacro:arg name="prefix" default="" />
   <xacro:arg name="use_sim" default="false" />
+  <!-- raw か jpeg。台数を積む構成では jpeg で経路の詰まりを避ける -->
+  <xacro:arg name="camera_format" default="raw" />
   <xacro:arg name="robot_name" default="sample_robot_1"/>
   <xacro:include filename="$(find sample_robot_description)/urdf/common.xacro"/>
@@ -169,5 +171,5 @@
     </inertial>
   </link>
-  <xacro:sample_robot_simulation prefix=""/>
+  <xacro:sample_robot_simulation prefix="" camera_format="$(arg camera_format)"/>
   <xacro:sample_robot_ros2_control name="$(arg robot_name)" use_sim="$(arg use_sim)"/>
 </robot>

File: colcon_ws/src/sample_robot_description/robots/sample_robot_2.urdf.xacro (robot description, xacro)
@@ -3,4 +3,6 @@
   <xacro:arg name="prefix" default="" />
   <xacro:arg name="use_sim" default="false" />
+  <!-- raw か jpeg。台数を積む構成では jpeg で経路の詰まりを避ける -->
+  <xacro:arg name="camera_format" default="raw" />
   <xacro:arg name="robot_name" default="sample_robot_2"/>
   <xacro:include filename="$(find sample_robot_description)/urdf/common.xacro"/>
@@ -169,5 +171,5 @@
     </inertial>
   </link>
-  <xacro:sample_robot_simulation prefix=""/>
+  <xacro:sample_robot_simulation prefix="" camera_format="$(arg camera_format)"/>
   <xacro:sample_robot_ros2_control name="$(arg robot_name)" use_sim="$(arg use_sim)"/>
 </robot>

File: colcon_ws/src/sample_robot_description/robots/sample_robot_3.urdf.xacro (robot description, xacro)
@@ -3,4 +3,6 @@
   <xacro:arg name="prefix" default="" />
   <xacro:arg name="use_sim" default="false" />
+  <!-- raw か jpeg。台数を積む構成では jpeg で経路の詰まりを避ける -->
+  <xacro:arg name="camera_format" default="raw" />
   <xacro:arg name="robot_name" default="sample_robot_3"/>
   <xacro:include filename="$(find sample_robot_description)/urdf/common.xacro"/>
@@ -169,5 +171,5 @@
     </inertial>
   </link>
-  <xacro:sample_robot_simulation prefix=""/>
+  <xacro:sample_robot_simulation prefix="" camera_format="$(arg camera_format)"/>
   <xacro:sample_robot_ros2_control name="$(arg robot_name)" use_sim="$(arg use_sim)"/>
 </robot>

File: colcon_ws/src/sample_robot_description/robots/sample_robot_4.urdf.xacro (robot description, xacro)
@@ -3,4 +3,6 @@
   <xacro:arg name="prefix" default="" />
   <xacro:arg name="use_sim" default="false" />
+  <!-- raw か jpeg。台数を積む構成では jpeg で経路の詰まりを避ける -->
+  <xacro:arg name="camera_format" default="raw" />
   <xacro:arg name="robot_name" default="sample_robot_4"/>
   <xacro:include filename="$(find sample_robot_description)/urdf/common.xacro"/>
@@ -169,5 +171,5 @@
     </inertial>
   </link>
-  <xacro:sample_robot_simulation prefix=""/>
+  <xacro:sample_robot_simulation prefix="" camera_format="$(arg camera_format)"/>
   <xacro:sample_robot_ros2_control name="$(arg robot_name)" use_sim="$(arg use_sim)"/>
 </robot>

File: colcon_ws/src/sample_robot_description/robots/sample_robot_5.urdf.xacro (robot description, xacro)
@@ -3,4 +3,6 @@
   <xacro:arg name="prefix" default="" />
   <xacro:arg name="use_sim" default="false" />
+  <!-- raw か jpeg。台数を積む構成では jpeg で経路の詰まりを避ける -->
+  <xacro:arg name="camera_format" default="raw" />
   <xacro:arg name="robot_name" default="sample_robot_5"/>
   <xacro:include filename="$(find sample_robot_description)/urdf/common.xacro"/>
@@ -169,5 +171,5 @@
     </inertial>
   </link>
-  <xacro:sample_robot_simulation prefix=""/>
+  <xacro:sample_robot_simulation prefix="" camera_format="$(arg camera_format)"/>
   <xacro:sample_robot_ros2_control name="$(arg robot_name)" use_sim="$(arg use_sim)"/>
 </robot>

File: colcon_ws/src/sample_robot_description/robots/sample_robot_6.urdf.xacro (robot description, xacro)
@@ -3,4 +3,6 @@
   <xacro:arg name="prefix" default="" />
   <xacro:arg name="use_sim" default="false" />
+  <!-- raw か jpeg。台数を積む構成では jpeg で経路の詰まりを避ける -->
+  <xacro:arg name="camera_format" default="raw" />
   <xacro:arg name="robot_name" default="sample_robot_6"/>
   <xacro:include filename="$(find sample_robot_description)/urdf/common.xacro"/>
@@ -169,5 +171,5 @@
     </inertial>
   </link>
-  <xacro:sample_robot_simulation prefix=""/>
+  <xacro:sample_robot_simulation prefix="" camera_format="$(arg camera_format)"/>
   <xacro:sample_robot_ros2_control name="$(arg robot_name)" use_sim="$(arg use_sim)"/>
 </robot>

File: colcon_ws/src/sample_robot_description/robots/sample_robot_7.urdf.xacro (robot description, xacro)
@@ -3,4 +3,6 @@
   <xacro:arg name="prefix" default="" />
   <xacro:arg name="use_sim" default="false" />
+  <!-- raw か jpeg。台数を積む構成では jpeg で経路の詰まりを避ける -->
+  <xacro:arg name="camera_format" default="raw" />
   <xacro:arg name="robot_name" default="sample_robot_7"/>
   <xacro:include filename="$(find sample_robot_description)/urdf/common.xacro"/>
@@ -169,5 +171,5 @@
     </inertial>
   </link>
-  <xacro:sample_robot_simulation prefix=""/>
+  <xacro:sample_robot_simulation prefix="" camera_format="$(arg camera_format)"/>
   <xacro:sample_robot_ros2_control name="$(arg robot_name)" use_sim="$(arg use_sim)"/>
 </robot>

File: colcon_ws/src/sample_robot_description/robots/sample_robot_8.urdf.xacro (robot description, xacro)
@@ -3,4 +3,6 @@
   <xacro:arg name="prefix" default="" />
   <xacro:arg name="use_sim" default="false" />
+  <!-- raw か jpeg。台数を積む構成では jpeg で経路の詰まりを避ける -->
+  <xacro:arg name="camera_format" default="raw" />
   <xacro:arg name="robot_name" default="sample_robot_8"/>
   <xacro:include filename="$(find sample_robot_description)/urdf/common.xacro"/>
@@ -169,5 +171,5 @@
     </inertial>
   </link>
-  <xacro:sample_robot_simulation prefix=""/>
+  <xacro:sample_robot_simulation prefix="" camera_format="$(arg camera_format)"/>
   <xacro:sample_robot_ros2_control name="$(arg robot_name)" use_sim="$(arg use_sim)"/>
 </robot>

File: colcon_ws/src/sample_robot_description/simulation/sample_robot.simulation.xacro (robot description, xacro)
@@ -8,4 +8,8 @@
     camera  -> /<robot>/<link>/image_raw   (sensor_msgs/Image)
                /<robot>/<link>/camera_info (sensor_msgs/CameraInfo)
+    camera (format=jpeg のとき)
+            -> /<robot>/<link>/image_raw/compressed (sensor_msgs/CompressedImage)
+               生画像の代わりに出る。720p の生画像は 1 枚 2.76 MB あり、
+               Unity から ros_tcp_endpoint への 1 本の TCP を詰まらせる
     contact -> /<robot>/<link>/contact_count   (std_msgs/Int32)
                /<robot>/<link>/contact         (std_msgs/Bool)
@@ -18,5 +22,5 @@
 -->
 <robot xmlns:xacro="http://ros.org/wiki/xacro">
-  <xacro:macro name="sample_robot_simulation" params="prefix">
+  <xacro:macro name="sample_robot_simulation" params="prefix camera_format:=raw">
     <!-- =============== Unity Simulator =============== -->
     <simulation>
@@ -68,4 +72,6 @@
           <width>960</width>
           <height>540</height>
+          <format>${camera_format}</format>
+          <quality>75</quality>
         </image>
         <clip>
@@ -81,4 +87,6 @@
           <width>180</width>
           <height>180</height>
+          <format>${camera_format}</format>
+          <quality>75</quality>
         </image>
         <clip>
